File: Kicad File/V-meter Magic eye.kicad_sch (KiCad schematic)
At the start: 48 parts, among them J1 15V, J2 VT138 socket, J3 BF IN, J4 VT138 socket, Q1 BUZ11, Q2 BC547, Q3 BC547, Q4 BC547, U1 NE555P, U5 VT138

Commit message: V 1.1
Inserito pdf dello schema elettrico PCB e montaggio componenti
Parts:
- added C12: 100nF, Capacitor_THT:C_Rect_L7.0mm_W2.5mm_P5.00mm, symbol Device:C
- D1: value 1N4007 -> RGP10M
- Q1: value BUZ11 -> IRFBG 30
- R14: value 16 1/2W -> 22 1W
- R9: value 47K -> 100K
Connections:
- net GND: now also C12.1
- net at Q3.3 (E), R10.2: now also C12.2
Other:
- note added: "D1 = Diodo Fast Switching 1000V 1A Peak30A qualsiasi con simili caratteristiche purchè Fast"
- note added: "L1 = bobina 40 spire filo 0,7mm avvolte su nucleo toroidale in ferrite dal diametro esterno di 20mm oppure 24mm (non è critica)"
- note added: "Ponticellare R14 con tensione di alimentazione inferiori a 12,6V non scendere comunque sotto i 12V"
- note removed: "L1 = bobina 60 spire filo 0,4mm avvolte su nucleo toroidale in ferrite dal diametro esterno di 20mm oppure 24mm (non è critica)"
- moved on the sheet: C6, R7, R8, RV2
